Commit message: 1.0m/s 版本

File: NUC_MID360/2_ROS2包_obstacle_detector/config/robot.urdf (robot description, URDF)
Before this commit: robot medical_robot, 4 links, 3 joints
Joints:
- joint livox_joint: origin xyz=0.10 0 0.37 rpy=0 0 0 -> xyz=0 0 0.33 rpy=0 0 0

Commit message: 29s版本 长焦镜头 到位采集滤波后再调整

File: NUC_MID360/2_ROS2包_obstacle_detector/config/robot.urdf (robot description, URDF)
Before this commit: robot medical_robot, 4 links, 3 joints
Links:
- added link arm; visual box size=0.30 0.28 0.37
Joints:
- added joint arm_joint: type fixed, parent base_link, child arm, origin xyz=0 0 0 rpy=0 0 0

Commit message: 比赛稳定代码快照 20261013

File: NUC_MID360/2_ROS2包_obstacle_detector/config/robot.urdf (robot description, URDF)
Before this commit: robot medical_robot, 5 links, 4 joints
Joints:
- joint livox_joint: origin xyz=0 0 0.33 rpy=0 0 0 -> xyz=0 0 0.35 rpy=0 0 0
